File: pcb/cad/gerenciador_de_bateria/gerenciador_de_bateria.kicad_pcb (KiCad board)
At the start: 2 copper layers, 51 parts, among them J1 Conn_01x02_Male, J12 Conn_01x02_Male, J14 Conn_01x03_Male, J2 Conn_01x02_Male, J20 Conn_01x02_Male, J21 Conn_01x03_Male, J3 Conn_01x03_Male, J9 Conn_01x02_Male, Q1 ZVN4106F, Q2 BC817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

Commit message: Inicio do layout de PCB
Parts:
- moved R5 32.9 mm to (147.3, 112.4)
- moved R4 25.7 mm to (163.8, 102.2)
- moved U1 24.1 mm to (135.3, 110.5), turned to -90 degrees
- moved R3 12.8 mm to (147.3, 109.2)
- moved C9 6.63 mm to (158.1, 106.0), turned to 90 degrees
- moved U4 3.20 mm to (159.5, 109.8)
Connections:
- U1 pad 1: (no net) -> /VIN
- U1 pad 2: (no net) -> Net-(R3-Pad1)
- U1 pad 3: (no net) -> Net-(R5-Pad1)
- U1 pad 4: (no net) -> unconnected-(U1-Pad4)
- U1 pad 5: (no net) -> GNDPWR
