File: pcb/cad/gerenciador_de_bateria_2.0/gerenciador_de_bateria_2.0.kicad_sch (KiCad schematic)
At the start: 35 parts, among them J1 Conn_01x01_Female, J2 Conn_01x01_Female, J3 Conn_01x01_Female, J4 Conn_01x01_Female, J5 Conn_01x02_Male, J6 Conn_01x01_Female, J7 Conn_01x01_Female, SW1 SW_Push, U1 MP2731, U2 USB_BQ25629

Commit message: Atualização da placa para gerenciamento de bateria, finalização do layout e roteamento
Parts:
- removed J1, J2, J3, J4, J6, J7, TERM1: Conn_01x01_Female, Connector_PinHeader_2.54mm:PinHeader_1x01_P2.54mm_Vertical, symbol Connector:Conn_01x01_Female
- added J1: Conn_01x05, Connector_PinHeader_2.54mm:PinHeader_1x05_P2.54mm_Vertical, symbol Connector_Generic:Conn_01x05
- added J2: Conn_01x02, Connector_PinHeader_2.54mm:PinHeader_1x02_P2.54mm_Vertical, symbol Connector_Generic:Conn_01x02
- SW1: footprint Button_Switch_THT:SW_PUSH_6mm -> Button_Switch_SMD:SW_SPST_B3U-1000P
Connections:
- net GNDPWR: now also J1.2 (Pin_2), J1.3 (Pin_3), J2.2 (Pin_2)
- net SYS: now also J1.4 (Pin_4)
- net BATT: now reaches C7.1, C9.2, U1.17 (BATT)
- net BATT: now also J1.1 (Pin_1)
- net VIN: now reaches C1.1, C12.1, U1.2 (IN), U2.1 (VBUS)
- net VIN: now also J2.1 (Pin_1)
- net TERM: now reaches R11.1
- net TERM: now also J1.5 (Pin_5)

Commit message: Revisão da PCB do gerenciador de bateria 2.0, corrigindo os GND que estavam flutuando e atualizando footprint de componentes que estavam errados
Parts:
- U2: footprint Connector_USB:USB_Micro-B_Amphenol_10118194_Horizontal -> Connector_USB:USB_Micro-B_Molex-105017-0001
Changed lines of the file:
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@@
       (effects (font (size 1.27 1.27)) hide)
     )
-    (property "Footprint" "Connector_USB:USB_Micro-B_Amphenol_10118194_Horizontal" (id 2) (at 85.979 69.342 0)
+    (property "Footprint" "Connector_USB:USB_Micro-B_Molex-105017-0001" (id 2) (at 85.979 69.342 0)
       (effects (font (size 1.27 1.27)) hide)
     )
@@
     )
     (path "/5c53f167-a398-4a5f-9744-88a876c8b5a1"
-      (reference "U2") (unit 1) (value "USB_BQ25629") (footprint "Connector_USB:USB_Micro-B_Amphenol_10118194_Horizontal")
-    )
-  )
+      (reference "U2") (unit 1) (value "USB_BQ25629") (footprint "Connector_USB:USB_Micro-B_Molex-105017-0001")
+    )
+  )
